File: dogooder.kicad_sch (KiCad schematic)
At the start: 37 parts, among them SW10 SW_PUSH, SW11 SW_PUSH, SW12 SW_PUSH, SW14 SW_PUSH, SW15 SW_PUSH, SW16 SW_PUSH, SW17 SW_PUSH, SW18 SW_PUSH, SW19 SW_PUSH, SW2 SW_PUSH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

Commit message: Add files via upload
Parts:
- removed SW?: SW_SPDT, symbol Switch:SW_SPDT
- added Bat+1, BatGND1: MountingHole_Pad, kbd:1pin_conn, symbol Mechanical:MountingHole_Pad
- added J1: AudioJack4dpb, kbd:MJ-4PP-9, symbol tokas_bp:AudioJack4dpb
- added SW_POWER1: SW_SPDT, Kailh:SPDT_C128955, symbol Switch:SW_SPDT
Connections:
- net raw: now reaches U1.14 (5V)
- net raw: now also SW_POWER1.3 (C)
- net data: now reaches U1.8 (PB09_A7_D7_RX)
- net data: now also J1.B
- new net BT+: Bat+1.1, SW_POWER1.2 (B)
- new net gnd: BatGND1.1, J1.C
- new net vcc: J1.D
Other:
- note added: "Battery Business"
- note added: "Useless TRRS"
Changed lines of the file:
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@@
+    (stroke (width 0) (type default) (color 0 0 0 0))
+  )
+  (polyline (pts (xy 204.47 162.56) (xy 204.47 109.22))
     (stroke (width 0) (type default) (color 0 0 0 0))
   )
@@
     (stroke (width 0) (type default) (color 0 0 0 0))
   )
+  (polyline (pts (xy 204.47 109.22) (xy 279.4 109.22))
+    (stroke (width 0) (type default) (color 0 0 0 0))
+  )
   (wire (pts (xy 95.25 48.26) (xy 95.25 63.5))
     (stroke (width 0) (type default) (color 0 0 0 0))
@@
     (stroke (width 0) (type default) (color 0 0 0 0))
   )
+  (polyline (pts (xy 279.4 109.22) (xy 279.4 162.56))
+    (stroke (width 0) (type default) (color 0 0 0 0))
+  )
   (wire (pts (xy 110.49 55.88) (xy 128.27 55.88))
     (stroke (width 0) (type default) (color 0 0 0 0))
@@
     (stroke (width 0) (type default) (color 0 0 0 0))
   )
+  (polyline (pts (xy 279.4 162.56) (xy 204.47 162.56))
+    (stroke (width 0) (type default) (color 0 0 0 0))
+  )
   (wire (pts (xy 110.49 71.12) (xy 128.27 71.12))
     (stroke (width 0) (type default) (color 0 0 0 0))
@@
   (wire (pts (xy 74.93 40.64) (xy 92.71 40.64))
     (stroke (width 0) (type default) (color 0 0 0 0))
+  )
+  (text "Battery Business" (at 220.98 116.84 0)
+    (effects (font (size 2.9972 2.9972)) (justify left bottom))
+  )
+  (text "Useless TRRS\n" (at 160.02 116.84 0)
+    (effects (font (size 2.9972 2.9972)) (justify left bottom))
+  )
+  (global_label "BT+" (shape input) (at 212.09 134.62 270) (fields_autoplaced)
+    (effects (font (size 1.27 1.27)) (justify right))
+    (property "Intersheet References" "${INTERSHEET_REFS}" (id 0) (at 0 3.81 0)
+      (effects (font (size 1.27 1.27)) hide)
+    )
+  )
+  (global_label "gnd" (shape input) (at 177.8 132.08 0) (fields_autoplaced)
+    (effects (font (size 1.27 1.27)) (justify left))
+    (property "Intersheet References" "${INTERSHEET_REFS}" (id 0) (at -11.43 80.01 0)
+      (effects (font (size 1.27 1.27)) hide)
+    )
   )
   (global_label "col4" (shape input) (at 198.12 52.07 0) (fields_autoplaced)
@@
     (property "Intersheet References" "${INTERSHEET_REFS}" (id 0) (at 22.225 9.525 0)
       (effects (font (size 1.27 1.27)) hide)
+    )
+  )
+  (global_label "raw" (shape input) (at 198.12 36.83 0) (fields_autoplaced)
+    (effects (font (size 1.27 1.27)) (justify left))
+    (property "Intersheet References" "${INTERSHEET_REFS}" (id 0) (at 203.7988 36.7506 0)
+      (effects (font (size 1.27 1.27)) (justify left) hide)
     )
   )
@@
     )
   )
+  (global_label "vcc" (shape input) (at 177.8 134.62 0) (fields_autoplaced)
+    (effects (font (size 1.27 1.27)) (justify left))
+    (property "Intersheet References" "${INTERSHEET_REFS}" (id 0) (at -11.43 80.01 0)
+      (effects (font (size 1.27 1.27)) hide)
+    )
+  )
   (global_label "row1" (shape input) (at 39.37 55.88 180) (fields_autoplaced)
     (effects (font (size 1.1938 1.1938)) (justify right))
@@
     )
   )
+  (global_label "gnd" (shape input) (at 245.11 140.97 180) (fields_autoplaced)
+    (effects (font (size 1.27 1.27)) (justify right))
+    (property "Intersheet References" "${INTERSHEET_REFS}" (id 0) (at 0 3.81 0)
+      (effects (font (size 1.27 1.27)) hide)
+    )
+  )
   (global_label "col5" (shape input) (at 198.12 55.88 0) (fields_autoplaced)
     (effects (font (size 1.1938 1.1938)) (justify left))
@@
     (effects (font (size 1.1938 1.1938)) (justify right))
     (property "Intersheet References" "${INTERSHEET_REFS}" (id 0) (at 15.875 1.905 0)
+      (effects (font (size 1.27 1.27)) hide)
+    )
+  )
+  (global_label "BT+" (shape input) (at 245.11 130.81 180) (fields_autoplaced)
+    (effects (font (size 1.27 1.27)) (justify right))
+    (property "Intersheet References" "${INTERSHEET_REFS}" (id 0) (at 0 3.81 0)
       (effects (font (size 1.27 1.27)) hide)
     )
@@
     (effects (font (size 1.1938 1.1938)) (justify right))
     (property "Intersheet References" "${INTERSHEET_REFS}" (id 0) (at 15.875 0.635 0)
+      (effects (font (size 1.27 1.27)) hide)
+    )
+  )
+  (global_label "data" (shape input) (at 198.12 59.69 0) (fields_autoplaced)
+    (effects (font (size 1.27 1.27)) (justify left))
+    (property "Intersheet References" "${INTERSHEET_REFS}" (id 0) (at 204.706 59.6106 0)
+      (effects (font (size 1.27 1.27)) (justify left) hide)
+    )
+  )
+  (global_label "data" (shape input) (at 177.8 129.54 0) (fields_autoplaced)
+    (effects (font (size 1.27 1.27)) (justify left))
+    (property "Intersheet References" "${INTERSHEET_REFS}" (id 0) (at 184.386 129.4606 0)
+      (effects (font (size 1.27 1.27)) (justify left) hide)
+    )
+  )
+  (global_label "raw" (shape input) (at 222.25 137.16 270) (fields_autoplaced)
+    (effects (font (size 1.27 1.27)) (justify right))
+    (property "Intersheet References" "${INTERSHEET_REFS}" (id 0) (at 0 3.81 0)
       (effects (font (size 1.27 1.27)) hide)
     )
@@
     (pin "2")
   )
+  (symbol (lib_id "Switch:SW_SPDT") (at 217.17 134.62 0) (unit 1)
+    (in_bom yes) (on_board yes)
+    (property "Reference" "SW_POWER1" (id 0) (at 217.17 127.381 0))
+    (property "Value" "SW_SPDT" (id 1) (at 217.17 129.6924 0))
+    (property "Footprint" "Kailh:SPDT_C128955" (id 2) (at 217.17 134.62 0)
+      (effects (font (size 1.27 1.27)) hide)
+    )
+    (property "Datasheet" "~" (id 3) (at 217.17 134.62 0)
+      (effects (font (size 1.27 1.27)) hide)
+    )
+    (pin "1")
+    (pin "2")
+    (pin "3")
+  )
   (symbol (lib_id "Device:D") (at 110.49 36.83 90) (unit 1)
     (in_bom yes) (on_board yes)
@@
     (pin "2")
   )
+  (symbol (lib_id "Mechanical:MountingHole_Pad") (at 245.11 128.27 0) (unit 1)
+    (in_bom yes) (on_board yes)
+    (property "Reference" "Bat+1" (id 0) (at 247.65 127.0254 0)
+      (effects (font (size 1.27 1.27)) (justify left))
+    )
+    (property "Value" "MountingHole_Pad" (id 1) (at 247.65 129.3368 0)
+      (effects (font (size 1.27 1.27)) (justify left))
+    )
+    (property "Footprint" "kbd:1pin_conn" (id 2) (at 245.11 128.27 0)
+      (effects (font (size 1.27 1.27)) hide)
+    )
+    (property "Datasheet" "~" (id 3) (at 245.11 128.27 0)
+      (effects (font (size 1.27 1.27)) hide)
+    )
+    (pin "1")
+  )
   (symbol (lib_id "kbd:SW_PUSH") (at 102.87 33.02 0) (unit 1)
     (in_bom yes) (on_board yes)
@@
     (pin "2")
   )
+  (symbol (lib_id "Mechanical:MountingHole_Pad") (at 245.11 138.43 0) (unit 1)
+    (in_bom yes) (on_board yes)
+    (property "Reference" "BatGND1" (id 0) (at 247.65 137.1854 0)
+      (effects (font (size 1.27 1.27)) (justify left))
+    )
+    (property "Value" "MountingHole_Pad" (id 1) (at 247.65 139.4968 0)
+      (effects (font (size 1.27 1.27)) (justify left))
+    )
+    (property "Footprint" "kbd:1pin_conn" (id 2) (at 245.11 138.43 0)
+      (effects (font (size 1.27 1.27)) hide)
+    )
+    (property "Datasheet" "~" (id 3) (at 245.11 138.43 0)
+      (effects (font (size 1.27 1.27)) hide)
+    )
+    (pin "1")
+  )
   (symbol (lib_id "kbd:SW_PUSH") (at 120.65 33.02 0) (unit 1)
     (in_bom yes) (on_board yes)
@@
     (pin "2")
   )
+  (symbol (lib_id "tokas_bp:AudioJack4dpb") (at 172.72 132.08 0) (unit 1)
+    (in_bom yes) (on_board yes)
+    (property "Reference" "J1" (id 0) (at 171.6278 123.825 0))
+    (property "Value" "AudioJack4dpb" (id 1) (at 171.6278 126.1364 0))
+    (property "Footprint" "kbd:MJ-4PP-9" (id 2) (at 172.72 132.08 0)
+      (effects (font (size 1.27 1.27)) hide)
+    )
+    (property "Datasheet" "~" (id 3) (at 172.72 132.08 0)
+      (effects (font (size 1.27 1.27)) hide)
+    )
+    (pin "A")
+    (pin "B")
+    (pin "C")
+    (pin "D")
+  )
   (symbol (lib_id "kbd:SW_PUSH") (at 49.53 63.5 0) (unit 1)
     (in_bom yes) (on_board yes)
@@
     (pin "2")
   )
-  (symbol (lib_id "Switch:SW_SPDT") (at 220.98 80.01 0) (unit 1)
-    (in_bom yes) (on_board yes) (fields_autoplaced)
-    (property "Reference" "SW?" (id 0) (at 220.98 72.39 0))
-    (property "Value" "SW_SPDT" (id 1) (at 220.98 74.93 0))
-    (property "Footprint" "" (id 2) (at 220.98 80.01 0)
-      (effects (font (size 1.27 1.27)) hide)
-    )
-    (property "Datasheet" "~" (id 3) (at 220.98 80.01 0)
-      (effects (font (size 1.27 1.27)) hide)
-    )
-    (pin "1")
-    (pin "2")
-    (pin "3")
-  )
   (symbol (lib_id "Device:D") (at 92.71 52.07 90) (unit 1)
     (in_bom yes) (on_board yes)
@@
       (reference "#PWR0104") (unit 1) (value "GND") (footprint "")
     )
+    (path "/61614cee-b370-4b29-a238-fc28a54dab71"
+      (reference "Bat+1") (unit 1) (value "MountingHole_Pad") (footprint "kbd:1pin_conn")
+    )
+    (path "/9fc7ac44-cb8c-4b0f-a19b-9c4d4ecd6ffd"
+      (reference "BatGND1") (unit 1) (value "MountingHole_Pad") (footprint "kbd:1pin_conn")
+    )
     (path "/e0130066-f120-45ab-8ca4-de7cd402c362"
       (reference "D1") (unit 1) (value "D") (footprint "Diode_SMD:D_1206_3216Metric")
@@
       (reference "D17") (unit 1) (value "D") (footprint "kbd:D3_TH")
     )
+    (path "/ae5b107f-9fec-448e-989b-4dc11f98914b"
+      (reference "J1") (unit 1) (value "AudioJack4dpb") (footprint "kbd:MJ-4PP-9")
+    )
     (path "/581488ee-fe1f-43d1-a23d-526666571191"
       (reference "RSW1") (unit 1) (value "SW_PUSH") (footprint "kbd:ResetSW_1side")
@@
       (reference "SW20") (unit 1) (value "SW_PUSH") (footprint "marbla:SW_MX_1u")
     )
-    (path "/e5889358-36b5-4652-9d71-4d4aa652a144"
-      (reference "SW?") (unit 1) (value "SW_SPDT") (footprint "")
+    (path "/5e3a9117-7414-4678-a10d-723b7e2d0990"
+      (reference "SW_POWER1") (unit 1) (value "SW_SPDT") (footprint "Kailh:SPDT_C128955")
     )
     (path "/2d7541bc-8639-470e-9c1a-39cf9d36180a"
